File: pcb/prueba kicad 2.kicad_pcb (KiCad board)
At the start: 2 copper layers, 50 x 25 mm, 9 parts, among them J1 +5V, J2 GND, J3 Battery Level, U1 ATtiny85-20PU

Commit message: Arreglar primer virtual wall que se echó la Trufa
Other:
- net class Default removed
